File: bluepill/hardware/c6021light.kicad_pcb (KiCad board)
At the start: 2 copper layers, 100 x 50 mm, 79 parts, among them J1 Barrel_Jack_Switch, J10 Conn_01x02, J11 Conn_01x02, J12 XpressNet, J2 Conn_02x04_Odd_Even, J3 Conn_02x16_Row_Letter_First, J30 Loconet, J31 Conn_01x02, J32 Conn_01x02, J4 Conn_01x02, J5 Grove I2C, J50 USB_B_Micro, J51 Conn_01x06, J52 Debug UART, J6 Conn_01x02, J7 Conn_01x02, J8 RJ45, Q30 BC337, Q31 BC547, Q32 BC547, SW1 SW_Push, U1 L7805, U10 SN75176, U2 L7808, U3 MCP2562, U30 LM393, U4 ISO1050DUB, U50 CH340C

Commit message: new PCB version
Parts:
- C30: footprint Capacitor_THT:C_Disc_D3.0mm_W1.6mm_P2.50mm -> Capacitor_THT:C_Rect_L7.0mm_W3.5mm_P2.50mm_P5.00mm
- J11: footprint Connector_PinHeader_2.54mm:PinHeader_1x02_P2.54mm_Vertical -> Connector_PinHeader_2.54mm:PinHeader_1x02_P2.54mm_Vertical_NB
- J31: value Conn_01x02 -> Conn_01x03; footprint Connector_PinHeader_2.54mm:PinHeader_1x02_P2.54mm_Vertical_NB -> Connector_PinHeader_2.54mm:PinHeader_1x03_P2.54mm_Vertical
- moved R40 3.32 mm to (172.5, 80.8)
- moved R35 3.25 mm to (169.4, 80.8)
- moved U30 3.15 mm to (159.3, 77.0)
- moved R37 3.10 mm to (166.2, 73.2)
- moved J31 2.50 mm to (189.3, 55.5), turned to 270 degrees
- moved C31 1.39 mm to (179.6, 76.8)
- moved D20 0.67 mm to (180.5, 63.9)
- moved D21 0.67 mm to (180.5, 59.4)
- moved TP2 0.55 mm to (114.2, 87.6)
- moved U2 0.55 mm to (114.2, 90.1)
- moved C4 0.53 mm to (118.7, 96.0)
- moved R41 0.51 mm to (188.2, 53.1)
- moved R42 0.47 mm to (188.2, 51.1)
- moved C3 0.41 mm to (118.7, 88.8)
- moved Q32 0.38 mm to (190.1, 59.2)
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Connections:
- J31 pad 1: Net-(J31-Pad1) -> +8V
- J31 pad 2: +12V -> Net-(J31-Pad2)
- Q31 pad 1: Net-(J31-Pad1) -> Net-(J31-Pad2)
- R42 pad 2: Net-(J31-Pad1) -> Net-(J31-Pad2)
Routing:
- net +8V: track 61.5 -> 190.3 mm, vias 2 -> 4
- net Net-(J31-Pad2): track 0.00 -> 17.8 mm, vias 0 -> 1
- net Net-(J31-Pad1): track 17.6 -> 0.00 mm, vias 1 -> 0
- net /LN_TX: track 47.0 -> 41.7 mm, vias 1 -> 0
- net +12V: track 173.1 -> 178.2 mm
- net Net-(J50-Pad2): track 15.6 -> 11.8 mm
- net Net-(R32-Pad2): track 26.4 -> 22.6 mm
- net Net-(R39-Pad1): track 16.4 -> 13.0 mm
- net Net-(Q30-Pad2): track 6.75 -> 9.95 mm
- net /RS485TxD: track 41.3 -> 38.7 mm
- net Net-(J30-Pad1): track 21.4 -> 18.8 mm
- net Net-(C30-Pad1): track 6.72 -> 8.77 mm
- net GND: track 246.5 -> 248.4 mm
- net /RS485ENA: track 35.7 -> 34.2 mm
- net /M_GO: track 23.3 -> 24.6 mm
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Other:
- board text added: "12V"
- board text added: "8V"
- board text added: "Damian Philipp 2021/03 Gerhard Bertelsmann"
- board text removed: "Damian Philipp 2021/01 Gerhard Bertelsmann"
